Commit message: Working to mirror chefbot for bender_sim

File: bender_model/bender_description/bender_base.urdf.xacro (robot description, xacro)
@@ -1 +1,187 @@
-<?xml version="1.0" ?>
+<?xml version="1.0"?>
+<!--
+/////////////////////////////////////////////////////////////////////
+This file outlines the physical dimensions of the Bender Robot.
+It takes input from the files common_properties_and_values.urdf.xacro
+and bender_model_properties.urdf.xacro.
+/////////////////////////////////////////////////////////////////////
+Bender is a robot with a rectangular body supported by two caster
+wheels in the front and back (modled by spheres with no friction)
+and two differential drive wheels modeled by cylinders.
+/////////////////////////////////////////////////////////////////////
+====================================================================
+Author: Connor Fuhrman
+Contact: cfuhrman at citadel dot edu
+Contact 2: connorfuhrman at outlook dot com
+====================================================================
+-->
+<robot name="bender" xmlns:xacro="http://ros.org/wiki/xacro">
+<!-- Include the parameters outlined in other files -->
+    <xacro:include filename="$(find bender_model)/bender_sim_parameters/bender_model_properties.urdf.xacro"/>
+    <xacro:include filename="$(find bender_model)/bender_sim_parameters/common_properties_and_values.urdf.xacro"/>
+<!-- Bender Bot -->
+  <!--  <xacro:macro name="kobuki"> -->
+    <!-- create the base_link -->
+    <link name="base_link">
+            <visual>
+              <geometry>
+                <box size="${base_len} ${base_wid} ${base_height}"/>
+              </geometry>
+              <xacro:property name="material_blue"/>
+            </visual>
+            <collision>
+                <geometry>
+                  <box size="${base_len} ${base_wid} ${base_height}"/>
+                </geometry>
+            </collision>
+            <xacro:default_inertial mass="1"/>
+    </link>
+    <joint name="base_footprint_joint" type="fixed">
+        <parent link="base_link"/>
+        <child link="base_footprint"/>
+        <axis xyz="0 0 0"/>
+        <origin xyz="0 0 ${-base_height}" rpy="0 0 0"/>
+    </joint>
+    <link name="base_footprint">
+        <visual>
+            <geometry>
+                <box size="0.001 0.001 0.001"/>
+            </geometry>
+        </visual>
+        <collision>
+            <geometry>
+                <box size="0.001 0.001 0.001"/>
+            </geometry>
+        </collision>
+        <xacro:default_inertial mass="0.001"/>
+    </link>
+    <xacro:macro name="caster" params="position reflect">
+        <joint name="${position}_wheel_joint" type="fixed">
+            <parent link="base_footprint"/>
+            <child link="${position}_wheel"/>
+            <axis xyz="0 0 1"/>
+            <origin xyz="${reflect*(base_wid/2)} 0 ${-1 * base_height}" rpy="${pi/2} 0 0"/>
+        </joint>
+        <link name="${position}_wheel">
+            <visual>
+                <geometry>
+                    <sphere radius="${caster_radius}"/>
+                </geometry>
+                <material name="white"/>
+            </visual>
+            <collision>
+                <geometry>
+                  <sphere radius="${caster_radius}"/>
+                </geometry>
+            </collision>
+            <xacro:default_inertial mass="0.5"/>
+        </link>
+    <!-- This block provides the simulator (Gazebo) with information on a few additional
+    physical properties. See http://gazebosim.org/tutorials/?tut=ros_urdf for more-->
+        <gazebo reference="${position}_wheel">
+            <mu1 value = "0.0"/>
+            <mu2 value = "0.0"/>
+            <kp  value = "10000000.0"/>
+            <kd  value = "1.0"/>
+            <material>Gazebo/Grey/</material>
+        </gazebo>
+    </xacro:macro>
+    <xacro:macro name="wheel" params="position reflect">
+        <joint name="${position}_wheel_joint" type="continuous">
+            <parent link="base_footprint"/>
+            <child link="${position}_wheel"/>
+            <axis xyz="0 0 1"/>
+            <origin xyz="0 ${reflect*(base_wid/2)} ${-1*base_height}" rpy="${-pi/2} 0 0"/>
+        </joint>
+        <link name="${position}_wheel">
+            <visual>
+                <geometry>
+                    <cylinder length = "${wheel_length}" radius="${wheel_radius}"/>
+                </geometry>
+                <material name="white"/>
+            </visual>
+            <collision>
+                <geometry>
+                  <cylinder length = "${wheel_length}" radius="${wheel_radius}"/>
+                </geometry>
+            </collision>
+            <xacro:default_inertial mass="0.5"/>
+        </link>
+    <!-- This block provides the simulator (Gazebo) with information on a few additional
+    physical properties. See http://gazebosim.org/tutorials/?tut=ros_urdf for more-->
+        <gazebo reference="${position}_wheel">
+            <mu1 value = "200.0"/>
+            <mu2 value = "100.0"/>
+            <kp value="1000000.0" />
+            <kd value="1.0" />
+            <fdir1 value="1 0 0"/>
+            <material>Gazebo/Grey/</material>
+        </gazebo>
+    <!-- This block connects the wheel joint to an actuator (motor), which informs both
+    simulation and visualization of the robot -->
+       <transmission name="${position}_wheel_trans">
+        <type>transmission_interface/SimpleTransmission</type>
+             <actuator name="${position}_wheel_motor">
+                  <mechanicalReduction>1</mechanicalReduction>
+             </actuator>
+         <joint name="${position}_wheel_joint">
+              <hardwareInterface>hardware_interface/VelocityJointInterface</hardwareInterface>
+         </joint>
+        </transmission>
+    </xacro:macro>
+    <!-- Creating the actual robot -->
+    <xacro:caster position="front" reflect="1"/>
+    <xacro:caster position="back"  reflect="-1"/>
+    <xacro:wheel  position="right" reflect="1"/>
+    <xacro:wheel  position="left"  reflect="-1"/>
+    <!-- Gazebo plugin for ROS Control -->
+    <gazebo>
+      <plugin name="gazebo_ros_control" filename="libgazebo_ros_control.so">
+        <robotNamespace>/</robotNamespace>
+      </plugin>
+    </gazebo>
+    <!-- Hokuyo Laser Senso -->
+    <link name="hokuyo_link">
+      <visual>
+        <origin xyz="0 0 0" rpy="0 0 0" />
+        <geometry>
+          <box size="${hokuyo_size} ${hokuyo_size} ${1.5*hokuyo_size}"/>
+        </geometry>
+        <material name="Blue" />
+      </visual>
+    </link>
+    <joint name="hokuyo_joint" type="fixed">
+      <origin xyz="${base_wid/2} 0 ${base_height+hokuyo_size/4}" rpy="0 0 0" />
+      <parent link="base_link"/>
+      <child link="hokuyo_link" />
+    </joint>
+    <gazebo reference="hokuyo_link">
+      <material>Gazebo/Blue</material>
+      <turnGravityOff>false</turnGravityOff>
+      <sensor type="ray" name="head_hokuyo_sensor">
+        <pose>${hokuyo_size/2} 0 0 0 0 0</pose>
+        <visualize>false</visualize>
+        <update_rate>40</update_rate>
+        <ray>
+          <scan>
+            <horizontal>
+              <samples>720</samples>
+              <resolution>1</resolution>
+              <min_angle>-1.570796</min_angle>
+              <max_angle>1.570796</max_angle>
+            </horizontal>
+          </scan>
+          <range>
+            <min>0.10</min>
+            <max>10.0</max>
+            <resolution>0.001</resolution>
+          </range>
+        </ray>
+        <plugin name="gazebo_ros_head_hokuyo_controller" filename="libgazebo_ros_laser.so">
+          <topicName>/scan</topicName>
+          <frameName>hokuyo_link</frameName>
+        </plugin>
+      </sensor>
+    </gazebo>
+ <!--   </xacro:macro> -->
+</robot>

File: bender_model/bender_sim_parameters/bender_model_properties.urdf.xacro (robot description, xacro)
@@ -1,2 +1,3 @@
+<?xml version="1.0"?>
 <!--
 =========================================================
@@ -5,5 +6,4 @@
 =========================================================
 -->
-<?xml version="1.0"?>
 <robot>
   <!--

File: bender_model/bender_sim_parameters/common_properties_and_values.urdf.xacro (robot description, xacro)
@@ -39,4 +39,14 @@
   <xacro:property name="update_rate" value="50"/>
   <xacro:property name="hokuyo_size" value="0.05"/>
+<!-- Default Inertial Values for Bender
+///////////////////////////////////////////////////////////////////
+-->
+<xacro:macro name="default_inertial" params="mass">
+    <inertial>
+      <mass value="${mass}" />
+      <inertia ixx="1.0" ixy="0.0" ixz="0.0"
+        iyy="1.0" iyz="0.0" izz="1.0" />
+    </inertial>
+</xacro:macro>
 <!-- Begin Colors:
 /////////////////////////////////////////////////////////////////////
