Commit message: Working simulation in rviz. Working to a simulation in gazebo.

File: bender_model/model.urdf.xacro (robot description, xacro)
@@ -5,11 +5,14 @@
     <xacro:property name="base_wid" value="0.80" />
     <xacro:property name="base_height" value="0.20" />
-    <xacro:property name="well_len" value="0.15" />
-    <xacro:property name="well_wid" value="0.15" />
-    <xacro:property name="well_height" value="0.15" />
     <xacro:property name="caster_length" value="0.10" />
     <xacro:property name="caster_radius" value="0.15" />
     <xacro:property name="wheel_length" value="0.10" />
     <xacro:property name="wheel_radius" value="0.15" />
+    <xacro:macro name="default_inertial" params="mass">
+        <inertial>
+          <mass value="${mass}" />
+          <inertia ixx="1.0" ixy="0.0" ixz="0.0" iyy="1.0" iyz="0.0" izz="1.0" />
+        </inertial>
+    </xacro:macro>
     <material name="white">
        <color rgba="1 1 1 1"/>
@@ -22,8 +25,15 @@
           <material name="white"/>
         </visual>
+        <collision>
+            <geometry>
+              <box size="${base_len} ${base_wid} ${base_height}"/>
+            </geometry>
+        </collision>
+        <xacro:default_inertial mass="10"/>
     </link>
-    <joint name="base_to_front_wheel" type="fixed">
+    <joint name="base_to_front_wheel" type="continuous">
         <parent link="base_link"/>
         <child link="front_wheel"/>
+        <axis xyz="0 0 1"/>
         <origin xyz="${base_wid/2} 0 ${-1*base_height}" rpy="${pi/2} 0 0"/>
     </joint>
@@ -35,8 +45,15 @@
             <material name="white"/>
         </visual>
+        <collision>
+            <geometry>
+              <cylinder length = "${caster_length}" radius="${caster_radius}"/>
+            </geometry>
+        </collision>
+        <xacro:default_inertial mass="2"/>
     </link>
-    <joint name="base_to_back_wheel" type="fixed">
+    <joint name="base_to_back_wheel" type="continuous">
         <parent link="base_link"/>
         <child link="back_wheel"/>
+        <axis xyz="0 0 1"/>
         <origin xyz="${-1*base_wid/2} 0 ${-1*base_height}" rpy="${pi/2} 0 0"/>
     </joint>
@@ -48,8 +65,15 @@
             <material name="white"/>
         </visual>
+        <collision>
+            <geometry>
+              <cylinder length = "${caster_length}" radius="${caster_radius}"/>
+            </geometry>
+        </collision>
+        <xacro:default_inertial mass="2"/>
     </link>
-    <joint name="base_to_right_wheel" type="fixed">
+    <joint name="base_to_right_wheel" type="continuous">
         <parent link="base_link"/>
         <child link="right_wheel"/>
+        <axis xyz="0 0 1"/>
         <origin xyz="0 ${-1*base_wid/2} ${-1*base_height}" rpy="${pi/2} 0 0"/>
     </joint>
@@ -61,8 +85,15 @@
             <material name="white"/>
         </visual>
+        <collision>
+            <geometry>
+              <cylinder length = "${wheel_length}" radius="${wheel_radius}"/>
+            </geometry>
+        </collision>
+        <xacro:default_inertial mass="5"/>
     </link>
-    <joint name="base_to_left_wheel" type="fixed">
+    <joint name="base_to_left_wheel" type="continuous">
         <parent link="base_link"/>
         <child link="left_wheel"/>
+        <axis xyz="0 0 1"/>
         <origin xyz="0 ${base_wid/2} ${-1*base_height}" rpy="${pi/2} 0 0"/>
     </joint>
@@ -74,4 +105,16 @@
             <material name="white"/>
         </visual>
+        <collision>
+            <geometry>
+              <cylinder length = "${wheel_length}" radius="${wheel_radius}"/>
+            </geometry>
+        </collision>
+        <xacro:default_inertial mass="5"/>
     </link>
+ <!-- Gazebo plugin for ROS Control -->
+    <gazebo>
+      <plugin name="gazebo_ros_control" filename="libgazebo_ros_control.so">
+        <robotNamespace>/</robotNamespace>
+      </plugin>
+    </gazebo>
 </robot>

Commit message: Gazebo model working except for the front and back casters for the robot.

File: bender_model/model.urdf.xacro (robot description, xacro)
@@ -16,5 +16,5 @@
     </xacro:macro>
     <material name="white">
-       <color rgba="1 1 1 1"/>
+       <color rgba="1 1 1 1.5"/>
     </material>
     <link name="base_link">
@@ -32,84 +32,91 @@
         <xacro:default_inertial mass="10"/>
     </link>
-    <joint name="base_to_front_wheel" type="continuous">
-        <parent link="base_link"/>
-        <child link="front_wheel"/>
-        <axis xyz="0 0 1"/>
-        <origin xyz="${base_wid/2} 0 ${-1*base_height}" rpy="${pi/2} 0 0"/>
-    </joint>
-    <link name="front_wheel">
-        <visual>
-            <geometry>
-                <cylinder length = "${caster_length}" radius="${caster_radius}"/>
-            </geometry>
-            <material name="white"/>
-        </visual>
-        <collision>
-            <geometry>
-              <cylinder length = "${caster_length}" radius="${caster_radius}"/>
-            </geometry>
-        </collision>
-        <xacro:default_inertial mass="2"/>
-    </link>
-    <joint name="base_to_back_wheel" type="continuous">
-        <parent link="base_link"/>
-        <child link="back_wheel"/>
-        <axis xyz="0 0 1"/>
-        <origin xyz="${-1*base_wid/2} 0 ${-1*base_height}" rpy="${pi/2} 0 0"/>
-    </joint>
-    <link name="back_wheel">
-        <visual>
-            <geometry>
-                 <cylinder length = "${caster_length}" radius="${caster_radius}"/>
-            </geometry>
-            <material name="white"/>
-        </visual>
-        <collision>
-            <geometry>
-              <cylinder length = "${caster_length}" radius="${caster_radius}"/>
-            </geometry>
-        </collision>
-        <xacro:default_inertial mass="2"/>
-    </link>
-    <joint name="base_to_right_wheel" type="continuous">
-        <parent link="base_link"/>
-        <child link="right_wheel"/>
-        <axis xyz="0 0 1"/>
-        <origin xyz="0 ${-1*base_wid/2} ${-1*base_height}" rpy="${pi/2} 0 0"/>
-    </joint>
-    <link name="right_wheel">
-        <visual>
-            <geometry>
-                <cylinder length = "${wheel_length}" radius="${wheel_radius}"/>
-            </geometry>
-            <material name="white"/>
-        </visual>
-        <collision>
-            <geometry>
-              <cylinder length = "${wheel_length}" radius="${wheel_radius}"/>
-            </geometry>
-        </collision>
-        <xacro:default_inertial mass="5"/>
-    </link>
-    <joint name="base_to_left_wheel" type="continuous">
-        <parent link="base_link"/>
-        <child link="left_wheel"/>
-        <axis xyz="0 0 1"/>
-        <origin xyz="0 ${base_wid/2} ${-1*base_height}" rpy="${pi/2} 0 0"/>
-    </joint>
-    <link name="left_wheel">
-        <visual>
-            <geometry>
-                <cylinder length = "${wheel_length}" radius="${wheel_radius}"/>
-            </geometry>
-            <material name="white"/>
-        </visual>
-        <collision>
-            <geometry>
-              <cylinder length = "${wheel_length}" radius="${wheel_radius}"/>
-            </geometry>
-        </collision>
-        <xacro:default_inertial mass="5"/>
-    </link>
+    <xacro:macro name="caster" params="position reflect">
+        <joint name="${position}_wheel_joint" type="continuous">
+            <parent link="base_link"/>
+            <child link="${position}_wheel"/>
+            <axis xyz="0 0 1"/>
+            <origin xyz="${reflect*base_wid/2} 0 ${-1 * base_height}" rpy="${pi/2} 0 0"/>
+        </joint>
+        <link name="${position}_wheel">
+            <visual>
+                <geometry>
+                    <cylinder length = "${caster_length}" radius="${caster_radius}"/>
+                </geometry>
+                <material name="white"/>
+            </visual>
+            <collision>
+                <geometry>
+                  <cylinder length = "${caster_length}" radius="${caster_radius}"/>
+                </geometry>
+            </collision>
+        </link>
+<!-- This block provides the simulator (Gazebo) with information on a few additional
+physical properties. See http://gazebosim.org/tutorials/?tut=ros_urdf for more-->
+        <gazebo reference="${position}_wheel">
+            <mu1 value = "200.0"/>
+            <mu2 value = "100.0"/>
+            <kp  value = "10000000.0"/>
+            <kd  value = "1.0"/>
+            <material>Gazebo/Grey/</material>
+        </gazebo>
+<!-- This block connects the wheel joint to an actuator (motor), which informs both
+   simulation and visualization of the robot -->
+       <transmission name="${position}_wheel_trans">
+        <type>transmission_interface/SimpleTransmission</type>
+             <actuator name="${position}_wheel_motor">
+                  <mechanicalReduction>1</mechanicalReduction>
+             </actuator>
+         <joint name="${position}_wheel_joint">
+              <hardwareInterface>VelocityJointInterface</hardwareInterface>
+         </joint>
+        </transmission>
+    </xacro:macro>
+    <xacro:macro name="wheel" params="position reflect">
+        <joint name="${position}_wheel_joint" type="continuous">
+            <parent link="base_link"/>
+            <child link="${position}_wheel"/>
+            <axis xyz="0 0 1"/>
+            <origin xyz="0 ${reflect*base_wid/2} ${-1*base_height}" rpy="${pi/2} 0 0"/>
+        </joint>
+        <link name="${position}_wheel">
+            <visual>
+                <geometry>
+                    <cylinder length = "${wheel_length}" radius="${wheel_radius}"/>
+                </geometry>
+                <material name="white"/>
+            </visual>
+            <collision>
+                <geometry>
+                  <cylinder length = "${wheel_length}" radius="${wheel_radius}"/>
+                </geometry>
+            </collision>
+            <xacro:default_inertial mass="5"/>
+        </link>
+<!-- This block provides the simulator (Gazebo) with information on a few additional
+physical properties. See http://gazebosim.org/tutorials/?tut=ros_urdf for more-->
+        <gazebo reference="${position}_wheel">
+            <mu1 value = "200.0"/>
+            <mu2 value = "100.0"/>
+            <kp  value = "10000000.0"/>
+            <kd  value = "1.0"/>
+            <material>Gazebo/Grey/</material>
+        </gazebo>
+<!-- This block connects the wheel joint to an actuator (motor), which informs both
+   simulation and visualization of the robot -->
+       <transmission name="${position}_wheel_trans">
+        <type>transmission_interface/SimpleTransmission</type>
+             <actuator name="${position}_wheel_motor">
+                  <mechanicalReduction>1</mechanicalReduction>
+             </actuator>
+         <joint name="${position}_wheel_joint">
+              <hardwareInterface>hardware_interface/VelocityJointInterface</hardwareInterface>
+         </joint>
+        </transmission>
+    </xacro:macro>
+    <xacro:caster position="front" reflect="1"/>
+    <xacro:caster position="back"  reflect="-1"/>
+    <xacro:wheel  position="right" reflect="1"/>
+    <xacro:wheel  position="left"  reflect="-1"/>
  <!-- Gazebo plugin for ROS Control -->
     <gazebo>

Commit message: Model simulated and moves front and back. Will not stear.

File: bender_model/model.urdf.xacro (robot description, xacro)
@@ -33,5 +33,5 @@
     </link>
     <xacro:macro name="caster" params="position reflect">
-        <joint name="${position}_wheel_joint" type="continuous">
+        <joint name="${position}_wheel_joint" type="fixed">
             <parent link="base_link"/>
             <child link="${position}_wheel"/>
@@ -55,21 +55,10 @@
 physical properties. See http://gazebosim.org/tutorials/?tut=ros_urdf for more-->
         <gazebo reference="${position}_wheel">
-            <mu1 value = "200.0"/>
-            <mu2 value = "100.0"/>
+            <mu1 value = "0.0"/>
+            <mu2 value = "0.0"/>
             <kp  value = "10000000.0"/>
             <kd  value = "1.0"/>
             <material>Gazebo/Grey/</material>
         </gazebo>
-<!-- This block connects the wheel joint to an actuator (motor), which informs both
-   simulation and visualization of the robot -->
-       <transmission name="${position}_wheel_trans">
-        <type>transmission_interface/SimpleTransmission</type>
-             <actuator name="${position}_wheel_motor">
-                  <mechanicalReduction>1</mechanicalReduction>
-             </actuator>
-         <joint name="${position}_wheel_joint">
-              <hardwareInterface>VelocityJointInterface</hardwareInterface>
-         </joint>
-        </transmission>
     </xacro:macro>
     <xacro:macro name="wheel" params="position reflect">
@@ -78,5 +67,5 @@
             <child link="${position}_wheel"/>
             <axis xyz="0 0 1"/>
-            <origin xyz="0 ${reflect*base_wid/2} ${-1*base_height}" rpy="${pi/2} 0 0"/>
+            <origin xyz="0 ${reflect*base_wid/2} ${-1*base_height}" rpy="${-pi/2} 0 0"/>
         </joint>
         <link name="${position}_wheel">

Commit message: bender model still only moves foward. Added LiDAR

File: bender_model/model.urdf.xacro (robot description, xacro)
@@ -9,4 +9,6 @@
     <xacro:property name="wheel_length" value="0.10" />
     <xacro:property name="wheel_radius" value="0.15" />
+    <xacro:property name="update_rate" value="50"/>
+    <xacro:property name="hokuyo_size" value="0.05"/>
     <xacro:macro name="default_inertial" params="mass">
         <inertial>
@@ -30,5 +32,5 @@
             </geometry>
         </collision>
-        <xacro:default_inertial mass="10"/>
+        <xacro:default_inertial mass="1"/>
     </link>
     <xacro:macro name="caster" params="position reflect">
@@ -37,10 +39,10 @@
             <child link="${position}_wheel"/>
             <axis xyz="0 0 1"/>
-            <origin xyz="${reflect*base_wid/2} 0 ${-1 * base_height}" rpy="${pi/2} 0 0"/>
+            <origin xyz="${reflect*(base_wid/2)} 0 ${-1 * base_height}" rpy="${pi/2} 0 0"/>
         </joint>
         <link name="${position}_wheel">
             <visual>
                 <geometry>
-                    <cylinder length = "${caster_length}" radius="${caster_radius}"/>
+                    <sphere radius="${caster_radius}"/>
                 </geometry>
                 <material name="white"/>
@@ -48,7 +50,8 @@
             <collision>
                 <geometry>
-                  <cylinder length = "${caster_length}" radius="${caster_radius}"/>
+                  <sphere radius="${caster_radius}"/>
                 </geometry>
             </collision>
+            <xacro:default_inertial mass="0.5"/>
         </link>
 <!-- This block provides the simulator (Gazebo) with information on a few additional
@@ -67,5 +70,5 @@
             <child link="${position}_wheel"/>
             <axis xyz="0 0 1"/>
-            <origin xyz="0 ${reflect*base_wid/2} ${-1*base_height}" rpy="${-pi/2} 0 0"/>
+            <origin xyz="0 ${reflect*(base_wid/2)} ${-1*base_height}" rpy="${-pi/2} 0 0"/>
         </joint>
         <link name="${position}_wheel">
@@ -81,5 +84,5 @@
                 </geometry>
             </collision>
-            <xacro:default_inertial mass="5"/>
+            <xacro:default_inertial mass="0.5"/>
         </link>
 <!-- This block provides the simulator (Gazebo) with information on a few additional
@@ -88,6 +91,7 @@
             <mu1 value = "200.0"/>
             <mu2 value = "100.0"/>
-            <kp  value = "10000000.0"/>
-            <kd  value = "1.0"/>
+            <kp value="1000000.0" />
+            <kd value="1.0" />
+            <fdir1 value="1 0 0"/>
             <material>Gazebo/Grey/</material>
         </gazebo>
@@ -114,3 +118,46 @@
       </plugin>
     </gazebo>
+<!-- Hokuyo Laser Senso -->
+    <link name="hokuyo_link">
+      <visual>
+        <origin xyz="0 0 0" rpy="0 0 0" />
+        <geometry>
+          <box size="${hokuyo_size} ${hokuyo_size} ${1.5*hokuyo_size}"/>
+        </geometry>
+        <material name="Blue" />
+      </visual>
+    </link>
+    <joint name="hokuyo_joint" type="fixed">
+      <origin xyz="${base_wid/2} 0 ${base_height+hokuyo_size/4}" rpy="0 0 0" />
+      <parent link="base_link"/>
+      <child link="hokuyo_link" />
+    </joint>
+    <gazebo reference="hokuyo_link">
+      <material>Gazebo/Blue</material>
+      <turnGravityOff>false</turnGravityOff>
+      <sensor type="ray" name="head_hokuyo_sensor">
+        <pose>${hokuyo_size/2} 0 0 0 0 0</pose>
+        <visualize>false</visualize>
+        <update_rate>40</update_rate>
+        <ray>
+          <scan>
+            <horizontal>
+              <samples>720</samples>
+              <resolution>1</resolution>
+              <min_angle>-1.570796</min_angle>
+              <max_angle>1.570796</max_angle>
+            </horizontal>
+          </scan>
+          <range>
+            <min>0.10</min>
+            <max>10.0</max>
+            <resolution>0.001</resolution>
+          </range>
+        </ray>
+        <plugin name="gazebo_ros_head_hokuyo_controller" filename="libgazebo_ros_laser.so">
+          <topicName>/scan</topicName>
+          <frameName>hokuyo_link</frameName>
+        </plugin>
+      </sensor>
+    </gazebo>
 </robot>
