Commit message: model has 4 wheels

File: bender_model/model.urdf.xacro (robot description, xacro)
@@ -34,43 +34,12 @@
         <xacro:default_inertial mass="1"/>
     </link>
-    <xacro:macro name="caster" params="position reflect">
-        <joint name="${position}_wheel_joint" type="fixed">
+    <xacro:macro name="front_wheel" params="position orient reflect">
+        <joint name="${position}_${orient}_wheel_joint" type="continuous">
             <parent link="base_link"/>
-            <child link="${position}_wheel"/>
+            <child link="${position}_${orient}_wheel"/>
             <axis xyz="0 0 1"/>
-            <origin xyz="${reflect*(base_wid/2)} 0 ${-1 * base_height}" rpy="${pi/2} 0 0"/>
+            <origin xyz="${base_len/2.5} ${reflect*(base_wid/2)} ${-1*base_height}" rpy="${-pi/2} 0 0"/>
         </joint>
-        <link name="${position}_wheel">
-            <visual>
-                <geometry>
-                    <sphere radius="${caster_radius}"/>
-                </geometry>
-                <material name="white"/>
-            </visual>
-            <collision>
-                <geometry>
-                  <sphere radius="${caster_radius}"/>
-                </geometry>
-            </collision>
-            <xacro:default_inertial mass="0.5"/>
-        </link>
-<!-- This block provides the simulator (Gazebo) with information on a few additional
-physical properties. See http://gazebosim.org/tutorials/?tut=ros_urdf for more-->
-        <gazebo reference="${position}_wheel">
-            <mu1 value = "0.0"/>
-            <mu2 value = "0.0"/>
-            <kp  value = "10000000.0"/>
-            <kd  value = "1.0"/>
-            <material>Gazebo/Grey/</material>
-        </gazebo>
-    </xacro:macro>
-    <xacro:macro name="wheel" params="position reflect">
-        <joint name="${position}_wheel_joint" type="continuous">
-            <parent link="base_link"/>
-            <child link="${position}_wheel"/>
-            <axis xyz="0 0 1"/>
-            <origin xyz="0 ${reflect*(base_wid/2)} ${-1*base_height}" rpy="${-pi/2} 0 0"/>
-        </joint>
-        <link name="${position}_wheel">
+        <link name="${position}_${orient}_wheel">
             <visual>
                 <geometry>
@@ -88,5 +57,5 @@
 <!-- This block provides the simulator (Gazebo) with information on a few additional
 physical properties. See http://gazebosim.org/tutorials/?tut=ros_urdf for more-->
-        <gazebo reference="${position}_wheel">
+        <gazebo reference="${position}_${orient}_wheel">
             <mu1 value = "200.0"/>
             <mu2 value = "100.0"/>
@@ -98,22 +67,66 @@
 <!-- This block connects the wheel joint to an actuator (motor), which informs both
    simulation and visualization of the robot -->
-       <transmission name="${position}_wheel_trans">
+       <transmission name="${position}_${orient}_wheel_trans">
         <type>transmission_interface/SimpleTransmission</type>
-             <actuator name="${position}_wheel_motor">
+             <actuator name="${position}_${orient}_wheel_motor">
                   <mechanicalReduction>1</mechanicalReduction>
              </actuator>
-         <joint name="${position}_wheel_joint">
+         <joint name="${position}_${orient}_wheel_joint">
               <hardwareInterface>hardware_interface/VelocityJointInterface</hardwareInterface>
          </joint>
         </transmission>
     </xacro:macro>
-    <xacro:caster position="front" reflect="1"/>
-    <xacro:caster position="back"  reflect="-1"/>
-    <xacro:wheel  position="right" reflect="1"/>
-    <xacro:wheel  position="left"  reflect="-1"/>
+    <xacro:macro name="back_wheel" params="position orient reflect">
+        <joint name="${position}_${orient}_wheel_joint" type="continuous">
+            <parent link="base_link"/>
+            <child link="${position}_${orient}_wheel"/>
+            <axis xyz="0 0 1"/>
+            <origin xyz="${-base_len/2.5} ${reflect*(base_wid/2)} ${-1*base_height}" rpy="${-pi/2} 0 0"/>
+        </joint>
+        <link name="${position}_${orient}_wheel">
+            <visual>
+                <geometry>
+                    <cylinder length = "${wheel_length}" radius="${wheel_radius}"/>
+                </geometry>
+                <material name="white"/>
+            </visual>
+            <collision>
+                <geometry>
+                  <cylinder length = "${wheel_length}" radius="${wheel_radius}"/>
+                </geometry>
+            </collision>
+            <xacro:default_inertial mass="0.5"/>
+        </link>
+    <!-- This block provides the simulator (Gazebo) with information on a few additional
+    physical properties. See http://gazebosim.org/tutorials/?tut=ros_urdf for more-->
+        <gazebo reference="${position}_${orient}_wheel">
+            <mu1 value = "200.0"/>
+            <mu2 value = "100.0"/>
+            <kp value="1000000.0" />
+            <kd value="1.0" />
+            <fdir1 value="1 0 0"/>
+            <material>Gazebo/Grey/</material>
+        </gazebo>
+    <!-- This block connects the wheel joint to an actuator (motor), which informs both
+    simulation and visualization of the robot -->
+       <transmission name="${position}_${orient}_wheel_trans">
+        <type>transmission_interface/SimpleTransmission</type>
+             <actuator name="${position}_${orient}_wheel_motor">
+                  <mechanicalReduction>1</mechanicalReduction>
+             </actuator>
+         <joint name="${position}_${orient}_wheel_joint">
+              <hardwareInterface>hardware_interface/VelocityJointInterface</hardwareInterface>
+         </joint>
+        </transmission>
+    </xacro:macro>
+    <xacro:front_wheel   orient="front" position="right" reflect="1"/>
+    <xacro:front_wheel    orient="front" position="left" reflect="-1"/>
+    <xacro:back_wheel   orient="back" position="right" reflect="1"/>
+    <xacro:back_wheel    orient="back" position="left" reflect="-1"/>
  <!-- Gazebo plugin for ROS Control -->
     <gazebo>
       <plugin name="gazebo_ros_control" filename="libgazebo_ros_control.so">
         <robotNamespace>/</robotNamespace>
+        <robotSimType>gazebo_ros_control/DefaultRobotHWSim</robotSimType>
       </plugin>
     </gazebo>

Commit message: Adding code from ROS Robotics Projects Ch 9/10

File: bender_model/model.urdf.xacro (robot description, xacro)
@@ -34,7 +34,26 @@
         <xacro:default_inertial mass="1"/>
     </link>
+    <joint name="base_footprint_joint" type="fixed">
+        <parent link="base_link"/>
+        <child link="base_footprint"/>
+        <axis xyz="0 0 0"/>
+        <origin xyz="0 0 ${-base_height}" rpy="0 0 0"/>
+    </joint>
+    <link name="base_footprint">
+        <visual>
+            <geometry>
+                <box size="0.001 0.001 0.001"/>
+            </geometry>
+        </visual>
+        <collision>
+            <geometry>
+                <box size="0.001 0.001 0.001"/>
+            </geometry>
+        </collision>
+        <xacro:default_inertial mass="0.001"/>
+    </link>
     <xacro:macro name="caster" params="position reflect">
         <joint name="${position}_wheel_joint" type="fixed">
-            <parent link="base_link"/>
+            <parent link="base_footprint"/>
             <child link="${position}_wheel"/>
             <axis xyz="0 0 1"/>
@@ -67,5 +86,5 @@
     <xacro:macro name="wheel" params="position reflect">
         <joint name="${position}_wheel_joint" type="continuous">
-            <parent link="base_link"/>
+            <parent link="base_footprint"/>
             <child link="${position}_wheel"/>
             <axis xyz="0 0 1"/>

Commit message: Changing bender model from Rev A to b. Creating initial model.

File: bender_model/model.urdf.xacro (robot description, xacro)
@@ -1,2 +1,4 @@
+<!-- Version A Commented out. Odometry does not give the correct
+lidar data representaion when robot rotates.
 <?xml version="1.0"?>
 <robot name="bender" xmlns:xacro="http://ros.org/wiki/xacro">
@@ -74,110 +76,113 @@
             <xacro:default_inertial mass="0.5"/>
         </link>
-<!-- This block provides the simulator (Gazebo) with information on a few additional
-physical properties. See http://gazebosim.org/tutorials/?tut=ros_urdf for more-->
-        <gazebo reference="${position}_wheel">
-            <mu1 value = "0.0"/>
-            <mu2 value = "0.0"/>
-            <kp  value = "10000000.0"/>
-            <kd  value = "1.0"/>
-            <material>Gazebo/Grey/</material>
+    <!- This block provides the simulator (Gazebo) with information on a few additional
+    physical properties. See http://gazebosim.org/tutorials/?tut=ros_urdf for more->
+            <gazebo reference="${position}_wheel">
+                <mu1 value = "0.0"/>
+                <mu2 value = "0.0"/>
+                <kp  value = "10000000.0"/>
+                <kd  value = "1.0"/>
+                <material>Gazebo/Grey/</material>
+            </gazebo>
+        </xacro:macro>
+        <xacro:macro name="wheel" params="position reflect">
+            <joint name="${position}_wheel_joint" type="continuous">
+                <parent link="base_footprint"/>
+                <child link="${position}_wheel"/>
+                <axis xyz="0 0 1"/>
+                <origin xyz="0 ${reflect*(base_wid/2)} ${-1*base_height}" rpy="${-pi/2} 0 0"/>
+            </joint>
+            <link name="${position}_wheel">
+                <visual>
+                    <geometry>
+                        <cylinder length = "${wheel_length}" radius="${wheel_radius}"/>
+                    </geometry>
+                    <material name="white"/>
+                </visual>
+                <collision>
+                    <geometry>
+                      <cylinder length = "${wheel_length}" radius="${wheel_radius}"/>
+                    </geometry>
+                </collision>
+                <xacro:default_inertial mass="0.5"/>
+            </link>
+    This block provides the simulator (Gazebo) with information on a few additional
+    physical properties. See http://gazebosim.org/tutorials/?tut=ros_urdf for more
+            <gazebo reference="${position}_wheel">
+                <mu1 value = "200.0"/>
+                <mu2 value = "100.0"/>
+                <kp value="1000000.0" />
+                <kd value="1.0" />
+                <fdir1 value="1 0 0"/>
+                <material>Gazebo/Grey/</material>
+            </gazebo>
+     This block connects the wheel joint to an actuator (motor), which informs both
+       simulation and visualization of the robot
+           <transmission name="${position}_wheel_trans">
+            <type>transmission_interface/SimpleTransmission</type>
+                 <actuator name="${position}_wheel_motor">
+                      <mechanicalReduction>1</mechanicalReduction>
+                 </actuator>
+             <joint name="${position}_wheel_joint">
+                  <hardwareInterface>hardware_interface/VelocityJointInterface</hardwareInterface>
+             </joint>
+            </transmission>
+        </xacro:macro>
+     Creating the actual robot
+        <xacro:caster position="front" reflect="1"/>
+        <xacro:caster position="back"  reflect="-1"/>
+        <xacro:wheel  position="right" reflect="1"/>
+        <xacro:wheel  position="left"  reflect="-1"/>
+      Gazebo plugin for ROS Control
+        <gazebo>
+          <plugin name="gazebo_ros_control" filename="libgazebo_ros_control.so">
+            <robotNamespace>/</robotNamespace>
+          </plugin>
         </gazebo>
-    </xacro:macro>
-    <xacro:macro name="wheel" params="position reflect">
-        <joint name="${position}_wheel_joint" type="continuous">
-            <parent link="base_footprint"/>
-            <child link="${position}_wheel"/>
-            <axis xyz="0 0 1"/>
-            <origin xyz="0 ${reflect*(base_wid/2)} ${-1*base_height}" rpy="${-pi/2} 0 0"/>
+     Hokuyo Laser Senso
+        <link name="hokuyo_link">
+          <visual>
+            <origin xyz="0 0 0" rpy="0 0 0" />
+            <geometry>
+              <box size="${hokuyo_size} ${hokuyo_size} ${1.5*hokuyo_size}"/>
+            </geometry>
+            <material name="Blue" />
+          </visual>
+        </link>
+        <joint name="hokuyo_joint" type="fixed">
+          <origin xyz="${base_wid/2} 0 ${base_height+hokuyo_size/4}" rpy="0 0 0" />
+          <parent link="base_link"/>
+          <child link="hokuyo_link" />
         </joint>
-        <link name="${position}_wheel">
-            <visual>
-                <geometry>
-                    <cylinder length = "${wheel_length}" radius="${wheel_radius}"/>
-                </geometry>
-                <material name="white"/>
-            </visual>
-            <collision>
-                <geometry>
-                  <cylinder length = "${wheel_length}" radius="${wheel_radius}"/>
-                </geometry>
-            </collision>
-            <xacro:default_inertial mass="0.5"/>
-        </link>
-<!-- This block provides the simulator (Gazebo) with information on a few additional
-physical properties. See http://gazebosim.org/tutorials/?tut=ros_urdf for more-->
-        <gazebo reference="${position}_wheel">
-            <mu1 value = "200.0"/>
-            <mu2 value = "100.0"/>
-            <kp value="1000000.0" />
-            <kd value="1.0" />
-            <fdir1 value="1 0 0"/>
-            <material>Gazebo/Grey/</material>
+        <gazebo reference="hokuyo_link">
+          <material>Gazebo/Blue</material>
+          <turnGravityOff>false</turnGravityOff>
+          <sensor type="ray" name="head_hokuyo_sensor">
+            <pose>${hokuyo_size/2} 0 0 0 0 0</pose>
+            <visualize>false</visualize>
+            <update_rate>40</update_rate>
+            <ray>
+              <scan>
+                <horizontal>
+                  <samples>720</samples>
+                  <resolution>1</resolution>
+                  <min_angle>-1.570796</min_angle>
+                  <max_angle>1.570796</max_angle>
+                </horizontal>
+              </scan>
+              <range>
+                <min>0.10</min>
+                <max>10.0</max>
+                <resolution>0.001</resolution>
+              </range>
+            </ray>
+            <plugin name="gazebo_ros_head_hokuyo_controller" filename="libgazebo_ros_laser.so">
+              <topicName>/scan</topicName>
+              <frameName>hokuyo_link</frameName>
+            </plugin>
+          </sensor>
         </gazebo>
-<!-- This block connects the wheel joint to an actuator (motor), which informs both
-   simulation and visualization of the robot -->
-       <transmission name="${position}_wheel_trans">
-        <type>transmission_interface/SimpleTransmission</type>
-             <actuator name="${position}_wheel_motor">
-                  <mechanicalReduction>1</mechanicalReduction>
-             </actuator>
-         <joint name="${position}_wheel_joint">
-              <hardwareInterface>hardware_interface/VelocityJointInterface</hardwareInterface>
-         </joint>
-        </transmission>
-    </xacro:macro>
-<!-- Creating the actual robot -->
-    <xacro:caster position="front" reflect="1"/>
-    <xacro:caster position="back"  reflect="-1"/>
-    <xacro:wheel  position="right" reflect="1"/>
-    <xacro:wheel  position="left"  reflect="-1"/>
- <!-- Gazebo plugin for ROS Control -->
-    <gazebo>
-      <plugin name="gazebo_ros_control" filename="libgazebo_ros_control.so">
-        <robotNamespace>/</robotNamespace>
-      </plugin>
-    </gazebo>
-<!-- Hokuyo Laser Senso -->
-    <link name="hokuyo_link">
-      <visual>
-        <origin xyz="0 0 0" rpy="0 0 0" />
-        <geometry>
-          <box size="${hokuyo_size} ${hokuyo_size} ${1.5*hokuyo_size}"/>
-        </geometry>
-        <material name="Blue" />
-      </visual>
-    </link>
-    <joint name="hokuyo_joint" type="fixed">
-      <origin xyz="${base_wid/2} 0 ${base_height+hokuyo_size/4}" rpy="0 0 0" />
-      <parent link="base_link"/>
-      <child link="hokuyo_link" />
-    </joint>
-    <gazebo reference="hokuyo_link">
-      <material>Gazebo/Blue</material>
-      <turnGravityOff>false</turnGravityOff>
-      <sensor type="ray" name="head_hokuyo_sensor">
-        <pose>${hokuyo_size/2} 0 0 0 0 0</pose>
-        <visualize>false</visualize>
-        <update_rate>40</update_rate>
-        <ray>
-          <scan>
-            <horizontal>
-              <samples>720</samples>
-              <resolution>1</resolution>
-              <min_angle>-1.570796</min_angle>
-              <max_angle>1.570796</max_angle>
-            </horizontal>
-          </scan>
-          <range>
-            <min>0.10</min>
-            <max>10.0</max>
-            <resolution>0.001</resolution>
-          </range>
-        </ray>
-        <plugin name="gazebo_ros_head_hokuyo_controller" filename="libgazebo_ros_laser.so">
-          <topicName>/scan</topicName>
-          <frameName>hokuyo_link</frameName>
-        </plugin>
-      </sensor>
-    </gazebo>
-</robot>
+    </robot>
+End version A.
+-->
+<!-- Begin Bender_Model Version B -->

Commit message: Odometry is working. Mapped environment

File: bender_model/model.urdf.xacro (robot description, xacro)
@@ -34,4 +34,5 @@
         <xacro:default_inertial mass="1"/>
     </link>
+<!--
     <joint name="base_footprint_joint" type="fixed">
         <parent link="base_link"/>
@@ -53,7 +54,8 @@
         <xacro:default_inertial mass="0.001"/>
     </link>
+-->
     <xacro:macro name="caster" params="position reflect">
         <joint name="${position}_wheel_joint" type="fixed">
-            <parent link="base_footprint"/>
+            <parent link="base_link"/>
             <child link="${position}_wheel"/>
             <axis xyz="0 0 1"/>
@@ -86,5 +88,5 @@
     <xacro:macro name="wheel" params="position reflect">
         <joint name="${position}_wheel_joint" type="continuous">
-            <parent link="base_footprint"/>
+            <parent link="base_link"/>
             <child link="${position}_wheel"/>
             <axis xyz="0 0 1"/>

Commit message: Navigation AMCL issue - laser scan.

File: bender_model/model.urdf.xacro (robot description, xacro)
@@ -11,4 +11,5 @@
     <xacro:property name="update_rate" value="50"/>
     <xacro:property name="hokuyo_size" value="0.05"/>
+    <!--robotBaseFrame>base_link</robotBaseFrame-->
     <xacro:macro name="default_inertial" params="mass">
         <inertial>
@@ -147,5 +148,5 @@
           <box size="${hokuyo_size} ${hokuyo_size} ${1.5*hokuyo_size}"/>
         </geometry>
-        <material name="Blue" />
+        <!--material name="Blue" /-->
       </visual>
     </link>
@@ -160,10 +161,11 @@
       <sensor type="ray" name="head_hokuyo_sensor">
         <pose>${hokuyo_size/2} 0 0 0 0 0</pose>
-        <visualize>false</visualize>
+        <!--visualize>false</visualize-->
+        <visualize>true</visualize>
         <update_rate>40</update_rate>
         <ray>
           <scan>
             <horizontal>
-              <samples>720</samples>
+              <samples>32</samples>
               <resolution>1</resolution>
               <min_angle>-1.570796</min_angle>
@@ -178,5 +180,5 @@
         </ray>
         <plugin name="gazebo_ros_head_hokuyo_controller" filename="libgazebo_ros_laser.so">
-          <topicName>/scan</topicName>
+          <topicName>scan</topicName>
           <frameName>hokuyo_link</frameName>
         </plugin>

Commit message: Working Nav - Gazebo URDF issue?

File: bender_model/model.urdf.xacro (robot description, xacro)
@@ -24,5 +24,5 @@
         <visual>
           <geometry>
-            <box size="${base_len} ${base_wid} ${base_height}"/>
+            <box size="${10*base_len} ${base_wid} ${base_height}"/>
           </geometry>
           <material name="white"/>
@@ -92,10 +92,10 @@
             <child link="${position}_wheel"/>
             <axis xyz="0 0 1"/>
-            <origin xyz="0 ${reflect*(base_wid/2)} ${-1*base_height}" rpy="${-pi/2} 0 0"/>
+            <origin xyz="0 ${reflect*(base_wid/2)} ${-1*base_height}" rpy="${pi/2} 0 0"/>
         </joint>
         <link name="${position}_wheel">
             <visual>
                 <geometry>
-                    <cylinder length = "${wheel_length}" radius="${wheel_radius}"/>
+                    <cylinder length = "${wheel_length}" radius="${2*wheel_radius}"/>
                 </geometry>
                 <material name="white"/>

Commit message: Model spawn correctly - edited world file that contained robot named robot. Robot named 'bender' now spawns

File: bender_model/model.urdf.xacro (robot description, xacro)
@@ -24,5 +24,5 @@
         <visual>
           <geometry>
-            <box size="${10*base_len} ${base_wid} ${base_height}"/>
+            <box size="${base_len} ${base_wid} ${base_height}"/>
           </geometry>
           <material name="white"/>
