Commit message: Gazebo model update. Add MATLAB file

File: bender_model/model.urdf.xacro (robot description, xacro)
@@ -11,5 +11,6 @@
     <xacro:property name="update_rate" value="50"/>
     <xacro:property name="hokuyo_size" value="0.05"/>
-    <!--robotBaseFrame>base_link</robotBaseFrame-->
+    <xacro:property name="camera_size" value="0.25"/>
+    <robotBaseFrame>base_link</robotBaseFrame>
     <xacro:macro name="default_inertial" params="mass">
         <inertial>
@@ -57,11 +58,11 @@
 -->
     <xacro:macro name="caster" params="position reflect">
-        <joint name="${position}_wheel_joint" type="fixed">
+        <joint name="${position}_caster_joint" type="fixed">
             <parent link="base_link"/>
-            <child link="${position}_wheel"/>
+            <child link="${position}_caster"/>
             <axis xyz="0 0 1"/>
             <origin xyz="${reflect*(base_wid/2)} 0 ${-1 * base_height}" rpy="${pi/2} 0 0"/>
         </joint>
-        <link name="${position}_wheel">
+        <link name="${position}_caster">
             <visual>
                 <geometry>
@@ -79,5 +80,5 @@
 <!-- This block provides the simulator (Gazebo) with information on a few additional
 physical properties. See http://gazebosim.org/tutorials/?tut=ros_urdf for more-->
-        <gazebo reference="${position}_wheel">
+        <gazebo reference="${position}_caster">
             <mu1 value = "0.0"/>
             <mu2 value = "0.0"/>
@@ -92,10 +93,10 @@
             <child link="${position}_wheel"/>
             <axis xyz="0 0 1"/>
-            <origin xyz="0 ${reflect*(base_wid/2)} ${-1*base_height}" rpy="${pi/2} 0 0"/>
+            <origin xyz="0 ${reflect*(base_wid/2)} ${-1*base_height}" rpy="${-pi/2} 0 0"/>
         </joint>
         <link name="${position}_wheel">
             <visual>
                 <geometry>
-                    <cylinder length = "${wheel_length}" radius="${2*wheel_radius}"/>
+                    <cylinder length = "${wheel_length}" radius="${wheel_radius}"/>
                 </geometry>
                 <material name="white"/>
@@ -141,4 +142,57 @@
       </plugin>
     </gazebo>
+<!-- Vision Camera -->
+    <link name="camera_link">
+        <visual>
+            <origin xyz="0 0 0" rpy="0 0 0" />
+            <geometry>
+                <box size="${camera_size} ${camera_size} ${camera_size}" />
+            </geometry>
+        </visual>
+    </link>
+    <joint name="camera_joint" type="fixed">
+      <origin xyz="0 0 ${4+base_height}" rpy="0 0 0" />
+      <parent link="base_link"/>
+      <child link="camera_link" />
+    </joint>
+    <gazebo reference="camera_link">
+      <sensor type="camera" name="camera">
+        <update_rate>30.0</update_rate>
+        <camera name="head">
+          <horizontal_fov>1.3962634</horizontal_fov>
+          <image>
+            <width>800</width>
+            <height>800</height>
+            <format>R8G8B8</format>
+          </image>
+          <clip>
+            <near>0.02</near>
+            <far>300</far>
+          </clip>
+          <noise>
+            <type>gaussian</type>
+            <!-- Noise is sampled independently per pixel on each frame.
+                 That pixel's noise value is added to each of its color
+                 channels, which at that point lie in the range [0,1]. -->
+            <mean>0.0</mean>
+            <stddev>0.007</stddev>
+          </noise>
+        </camera>
+        <plugin name="camera_controller" filename="libgazebo_ros_camera.so">
+          <alwaysOn>true</alwaysOn>
+          <updateRate>0.0</updateRate>
+          <cameraName>camera</cameraName>
+          <imageTopicName>image_raw</imageTopicName>
+          <cameraInfoTopicName>camera_info</cameraInfoTopicName>
+          <frameName>camera_link</frameName>
+          <hackBaseline>0.07</hackBaseline>
+          <distortionK1>0.0</distortionK1>
+          <distortionK2>0.0</distortionK2>
+          <distortionK3>0.0</distortionK3>
+          <distortionT1>0.0</distortionT1>
+          <distortionT2>0.0</distortionT2>
+        </plugin>
+      </sensor>
+    </gazebo>
 <!-- Hokuyo Laser Senso -->
     <link name="hokuyo_link">
@@ -163,5 +217,5 @@
         <!--visualize>false</visualize-->
         <visualize>true</visualize>
-        <update_rate>50</update_rate>
+        <update_rate>30</update_rate>
         <ray>
           <scan>

Commit message: Gazebo sim works with white lines and grass. Note that /grass needs to be placed into ~/.gazebo/models

File: bender_model/model.urdf.xacro (robot description, xacro)
@@ -152,5 +152,5 @@
     </link>
     <joint name="camera_joint" type="fixed">
-      <origin xyz="0 0 ${4+base_height}" rpy="0 0 0" />
+      <origin xyz="0 0 ${1+base_height}" rpy="0 0 0" />
       <parent link="base_link"/>
       <child link="camera_link" />

Commit message: Working image transform. Adding GPS to Gazebo. Modify move_base to work without map.

File: bender_model/model.urdf.xacro (robot description, xacro)
@@ -2,7 +2,7 @@
 <robot name="bender" xmlns:xacro="http://ros.org/wiki/xacro">
     <xacro:property name="pi" value="3.141592653589794" />
-    <xacro:property name="base_len" value="0.89" />
-    <xacro:property name="base_wid" value="0.80" />
-    <xacro:property name="base_height" value="0.20" />
+    <xacro:property name="base_len" value="0.90" />
+    <xacro:property name="base_wid" value="0.56" />
+    <xacro:property name="base_height" value="0.71" />
     <xacro:property name="caster_length" value="0.10" />
     <xacro:property name="caster_radius" value="0.15" />
@@ -12,4 +12,5 @@
     <xacro:property name="hokuyo_size" value="0.05"/>
     <xacro:property name="camera_size" value="0.25"/>
+    <xacro:property name="cam_pitch" value="${-pi/6}"/>
     <robotBaseFrame>base_link</robotBaseFrame>
     <xacro:macro name="default_inertial" params="mass">
@@ -62,5 +63,5 @@
             <child link="${position}_caster"/>
             <axis xyz="0 0 1"/>
-            <origin xyz="${reflect*(base_wid/2)} 0 ${-1 * base_height}" rpy="${pi/2} 0 0"/>
+            <origin xyz="${reflect*(base_wid/2)} 0 ${-0.5 * base_height}" rpy="${pi/2} 0 0"/>
         </joint>
         <link name="${position}_caster">
@@ -93,5 +94,5 @@
             <child link="${position}_wheel"/>
             <axis xyz="0 0 1"/>
-            <origin xyz="0 ${reflect*(base_wid/2)} ${-1*base_height}" rpy="${-pi/2} 0 0"/>
+            <origin xyz="0 ${reflect*(base_wid/2)} ${-0.5*base_height}" rpy="${-pi/2} 0 0"/>
         </joint>
         <link name="${position}_wheel">
@@ -142,4 +143,18 @@
       </plugin>
     </gazebo>
+<!-- Gazebo plugin for GPS data -->
+    <gazebo>
+        <plugin name="gps_controller" filename="libhector_gazebo_ros_gps.so">
+            <alwayson>true</alwayson>
+            <updaterate>1.0</updaterate>
+            <bodyname>base_link</bodyname>
+            <topicname>/fix</topicname>
+            <velocitytopicname>/fix_velocity</velocitytopicname>
+            <drift>5.0 5.0 5.0</drift>
+            <gaussiannoise>0.1 0.1 0.1</gaussiannoise>
+            <velocitydrift>0 0 0</velocitydrift>
+            <velocitygaussiannoise>0.1 0.1 0.1</velocitygaussiannoise>
+        </plugin>
+    </gazebo>
 <!-- Vision Camera -->
     <link name="camera_link">
@@ -152,5 +167,5 @@
     </link>
     <joint name="camera_joint" type="fixed">
-      <origin xyz="0 0 ${1+base_height}" rpy="0 0 0" />
+      <origin xyz="0 0 ${1+base_height}" rpy="0 ${-cam_pitch} 0" />
       <parent link="base_link"/>
       <child link="camera_link" />
@@ -162,7 +177,7 @@
           <horizontal_fov>1.3962634</horizontal_fov>
           <image>
-            <width>640</width>
+            <width>752</width>
             <height>480</height>
-            <format>R8G8B8</format>
+            <format>L8</format>
           </image>
           <clip>
@@ -170,12 +185,12 @@
             <far>300</far>
           </clip>
-          <noise>
+          <!--noise>
             <type>gaussian</type>
-            <!-- Noise is sampled independently per pixel on each frame.
+            < Noise is sampled independently per pixel on each frame.
                  That pixel's noise value is added to each of its color
-                 channels, which at that point lie in the range [0,1]. -->
+                 channels, which at that point lie in the range [0,1]. >
             <mean>0.0</mean>
             <stddev>0.007</stddev>
-          </noise>
+          </noise-->
         </camera>
         <plugin name="camera_controller" filename="libgazebo_ros_camera.so">
@@ -215,6 +230,6 @@
       <sensor type="ray" name="head_hokuyo_sensor">
         <pose>${hokuyo_size/2} 0 0 0 0 0</pose>
-        <!--visualize>false</visualize-->
-        <visualize>true</visualize>
+        <visualize>false</visualize>
+        <!--visualize>true</visualize-->
         <update_rate>30</update_rate>
         <ray>

Commit message: Added IMU to Gazebo model

File: bender_model/model.urdf.xacro (robot description, xacro)
@@ -11,4 +11,5 @@
     <xacro:property name="update_rate" value="50"/>
     <xacro:property name="hokuyo_size" value="0.05"/>
+    <xacro:property name="imu_size" value="0.025"/>
     <xacro:property name="camera_size" value="0.25"/>
     <xacro:property name="cam_pitch" value="${-pi/6}"/>
@@ -221,5 +222,5 @@
     </link>
     <joint name="hokuyo_joint" type="fixed">
-      <origin xyz="${base_wid/2} 0 ${base_height+hokuyo_size/4}" rpy="0 0 0" />
+      <origin xyz="${base_wid/2} 0 ${base_height*0.55}" rpy="0 0 0" />
       <parent link="base_link"/>
       <child link="hokuyo_link" />
@@ -254,3 +255,38 @@
       </sensor>
     </gazebo>
+<!-- Gazebo IMU -->
+    <link name="imu_link">
+      <visual>
+        <origin xyz="0 0 0" rpy="0 0 0" />
+        <geometry>
+          <box size="${imu_size} ${imu_size} ${imu_size}"/>
+        </geometry>
+        <!--material name="Blue" /-->
+      </visual>
+    </link>
+    <joint name="imu_joint" type="fixed">
+      <origin xyz="0 ${-1*base_wid/2} ${base_height*0.55}" rpy="0 0 0" />
+      <parent link="base_link"/>
+      <child link="imu_link" />
+    </joint>
+    <gazebo reference="imu_link">
+    <material>Gazebo/Red</material>
+      <gravity>true</gravity>
+      <sensor name="imu_sensor" type="imu">
+        <always_on>true</always_on>
+        <update_rate>100</update_rate>
+        <visualize>true</visualize>
+        <topic>"__default_topic__"/</topic>
+        <plugin filename="libgazebo_ros_imu_sensor.so" name="imu_plugin">
+          <topicName>imu</topicName>
+          <bodyName>imu_link</bodyName>
+          <updateRateHZ>10.0</updateRateHZ>
+          <gaussianNoise>0.0</gaussianNoise>
+          <xyzOffset>0 0 0</xyzOffset>
+          <rpyOffset>0 0 0</rpyOffset>
+          <frameName>imu_link</frameName>
+        </plugin>
+        <pose>0 0 0 0 0 0</pose>
+      </sensor>
+    </gazebo>
 </robot>

Commit message: EKF filter realized in Gazebo through robot_localization package. Working adding GPS to Bender Gazebo model

File: bender_model/model.urdf.xacro (robot description, xacro)
@@ -290,3 +290,40 @@
       </sensor>
     </gazebo>
+<!-- Gazebo GPS -->
+    <link name="gps_link">
+      <visual>
+        <origin xyz="0 0 0" rpy="0 0 0" />
+        <geometry>
+          <box size="${imu_size} ${imu_size} ${imu_size}"/>
+        </geometry>
+        <!--material name="Blue" /-->
+      </visual>
+    </link>
+    <joint name="gps_joint" type="fixed">
+      <origin xyz="0 ${1*base_wid/2} ${base_height*0.55}" rpy="0 0 0" />
+      <parent link="base_link"/>
+      <child link="gps_link" />
+    </joint>
+    <gazebo>
+        <plugin name="gazebo_ros_gps" filename="libhector_gazebo_ros_gps.so">
+            <updateRate>4.0</updateRate>
+            <bodyName>gps</bodyName>
+            <frameId>gps</frameId>
+            <topicName>/gps/fix</topicName>
+            <velocityTopicName>/gps/fix_velocity</velocityTopicName>
+            <referenceLatitude>-30.06022459407145675</referenceLatitude>
+            <referenceLongitude>-51.173913575780311191</referenceLongitude>
+            <referenceHeading>90</referenceHeading>
+            <referenceAltitude>10</referenceAltitude>
+            <offset>0 0 0</offset>
+            <drift>0.001 0.001 0.001</drift>
+            <gaussianNoise>0.05 0.05 0.05</gaussianNoise>
+            <velocityDrift>0.001 0.001 0.001</velocityDrift>
+            <velocityGaussianNoise>0.5 0.5 0.5</velocityGaussianNoise>
+    <!--                <drift>0.001 0.001 0.001</drift>-->
+    <!--                <gaussianNoise>0.01 0.01 0.01</gaussianNoise>-->
+    <!--                <velocityDrift>0 0 0</velocityDrift>-->
+    <!--                <velocityGaussianNoise>0.05 0.05 0.05</velocityGaussianNoise>-->
+        </plugin>
+    </gazebo>
 </robot>
